File: OpAmp_Inverting_DualSupply.sch (KiCad schematic (older format))
At the start: 11 parts, among them P201 CONN_2, P202 CONN_2, U201 TL071

Commit message: unknown updates
unknown updates
Parts:
- C201, C202: symbol CP1 -> CP1-RESCUE-SingleOpAmp_Inverting_DualSupply
- R201, R202, R203: symbol R -> R-RESCUE-SingleOpAmp_Inverting_DualSupply
Changed lines of the file:
@@
 EESchema Schematic File Version 2
+LIBS:SingleOpAmp_Inverting_DualSupply-rescue
 LIBS:power
 LIBS:device
@@
 LIBS:memory
 LIBS:xilinx
-LIBS:special
 LIBS:microcontrollers
 LIBS:dsp
@@
 LIBS:diy_ics
 LIBS:SingleOpAmp_Inverting_DualSupply-cache
-EELAYER 27 0
+EELAYER 25 0
 EELAYER END
 $Descr A4 11693 8268
@@
 $EndDescr
 $Comp
-L R R202
+L R-RESCUE-SingleOpAmp_Inverting_DualSupply R202
 U 1 1 532D87D7
 P 6500 6100
@@
 $EndComp
 $Comp
-L R R201
+L R-RESCUE-SingleOpAmp_Inverting_DualSupply R201
 U 1 1 532D87DD
 P 4750 4850
@@
 $EndComp
 $Comp
-L GND #PWR02
-U 1 1 532D8807
-P 4650 2750
-F 0 "#PWR02" H 4650 2750 30  0001 C CNN
-F 1 "GND" H 4650 2680 30  0001 C CNN
-F 2 "" H 4650 2750 60  0000 C CNN
-F 3 "" H 4650 2750 60  0000 C CNN
-	1    4650 2750
-	1    0    0    -1
-$EndComp
-$Comp
 L VCC #PWR03
 U 1 1 532D880D
@@
 	1    0    0    -1
 $EndComp
-$Comp
-L GND #PWR04
-U 1 1 532D8813
-P 3500 5250
-F 0 "#PWR04" H 3500 5250 30  0001 C CNN
-F 1 "GND" H 3500 5180 30  0001 C CNN
-F 2 "" H 3500 5250 60  0000 C CNN
-F 3 "" H 3500 5250 60  0000 C CNN
-	1    3500 5250
-	1    0    0    -1
-$EndComp
 Wire Wire Line
 	7000 4750 8650 4750
@@
 Wire Wire Line
 	8450 4950 8450 5250
-$Comp
-L GND #PWR05
-U 1 1 532D883C
-P 8450 5250
-F 0 "#PWR05" H 8450 5250 30  0001 C CNN
-F 1 "GND" H 8450 5180 30  0001 C CNN
-F 2 "" H 8450 5250 60  0000 C CNN
-F 3 "" H 8450 5250 60  0000 C CNN
-	1    8450 5250
-	1    0    0    -1
-$EndComp
 $Comp
 L BATTERY BT201
@@
 	4650 2550 4150 2550
 Connection ~ 4150 2550
-$Comp
-L GND #PWR06
-U 1 1 532D89A8
-P 5600 4650
-F 0 "#PWR06" H 5600 4650 30  0001 C CNN
-F 1 "GND" H 5600 4580 30  0001 C CNN
-F 2 "" H 5600 4650 60  0000 C CNN
-F 3 "" H 5600 4650 60  0000 C CNN
-	1    5600 4650
-	0    1    1    0
-$EndComp
 Text Notes 5100 2100 0    60   ~ 0
 TWO 9V BATTERIES ARE USED TO GENERATE THE VCC AND VEE OF +9V AND -9V. \nTHE BATTERY GND LINES ARE CONNECTED TOGETHER.
-$Comp
-L GND #PWR07
-U 1 1 532D9158
-P 3250 2650
-F 0 "#PWR07" H 3250 2650 30  0001 C CNN
-F 1 "GND" H 3250 2580 30  0001 C CNN
-F 2 "" H 3250 2650 60  0000 C CNN
-F 3 "" H 3250 2650 60  0000 C CNN
-	1    3250 2650
-	1    0    0    -1
-$EndComp
 Wire Wire Line
 	3000 2750 3000 2350
@@
 $EndComp
 $Comp
-L CP1 C201
+L CP1-RESCUE-SingleOpAmp_Inverting_DualSupply C201
 U 1 1 532D9261
 P 3000 2150
+AR Path="/532D9261" Ref="C201"  Part="1"
+AR Path="/532D86CE/532D9261" Ref="C201"  Part="1"
 F 0 "C201" H 3050 2250 50  0000 L CNN
 F 1 "100u" H 3050 2050 50  0000 L CNN
@@
 $EndComp
 $Comp
-L CP1 C202
+L CP1-RESCUE-SingleOpAmp_Inverting_DualSupply C202
 U 1 1 532D9270
 P 3000 2950
+AR Path="/532D9270" Ref="C202"  Part="1"
+AR Path="/532D86CE/532D9270" Ref="C202"  Part="1"
 F 0 "C202" H 3050 3050 50  0000 L CNN
 F 1 "100u" H 3050 2850 50  0000 L CNN
@@
 	6800 5150 6800 5250
 $Comp
-L R R203
+L R-RESCUE-SingleOpAmp_Inverting_DualSupply R203
 U 1 1 532DE079
 P 7350 5500
@@
 Text Notes 7000 4250 0    60   ~ 0
 GAIN = A(v) = VOUT/VIN = -RF/RIN
+$Comp
+L GND #PWR?
+U 1 1 55C79976
+P 3500 5250
+F 0 "#PWR?" H 3500 5000 50  0001 C CNN
+F 1 "GND" H 3500 5100 50  0000 C CNN
+F 2 "" H 3500 5250 60  0000 C CNN
+F 3 "" H 3500 5250 60  0000 C CNN
+	1    3500 5250
+	1    0    0    -1
+$EndComp
+$Comp
+L GND #PWR?
+U 1 1 55C799AB
+P 8450 5250
+F 0 "#PWR?" H 8450 5000 50  0001 C CNN
+F 1 "GND" H 8450 5100 50  0000 C CNN
+F 2 "" H 8450 5250 60  0000 C CNN
+F 3 "" H 8450 5250 60  0000 C CNN
+	1    8450 5250
+	1    0    0    -1
+$EndComp
+$Comp
+L GND #PWR?
+U 1 1 55C799E0
+P 4650 2750
+F 0 "#PWR?" H 4650 2500 50  0001 C CNN
+F 1 "GND" H 4650 2600 50  0000 C CNN
+F 2 "" H 4650 2750 60  0000 C CNN
+F 3 "" H 4650 2750 60  0000 C CNN
+	1    4650 2750
+	1    0    0    -1
+$EndComp
+$Comp
+L GND #PWR?
+U 1 1 55C79A2B
+P 3250 2650
+F 0 "#PWR?" H 3250 2400 50  0001 C CNN
+F 1 "GND" H 3250 2500 50  0000 C CNN
+F 2 "" H 3250 2650 60  0000 C CNN
+F 3 "" H 3250 2650 60  0000 C CNN
+	1    3250 2650
+	1    0    0    -1
+$EndComp
+$Comp
+L GND #PWR?
+U 1 1 55C79A7D
+P 5600 4650
+F 0 "#PWR?" H 5600 4400 50  0001 C CNN
+F 1 "GND" H 5600 4500 50  0000 C CNN
+F 2 "" H 5600 4650 60  0000 C CNN
+F 3 "" H 5600 4650 60  0000 C CNN
+	1    5600 4650
+	0    1    1    0
+$EndComp
 $EndSCHEMATC
